File: Board_760032v2.brd (EAGLE design)
At the start: 111.3 x 82.8 mm, 17 parts, among them J1 1X2-3.5MM, X1 JST-XH-04-PIN-LONG-PAD, X2 JST-XH-04-PIN-LONG-PAD, X3 JST-XH-04-PIN-LONG-PAD, X4 JST-XH-03-PIN-LONG-PAD, X5 btn0, X6 JST-XH-04-PIN-LONG-PAD, X8 JST-XH-02-PIN-LONG-PAD, X9 JST-XH-04-PIN-LONG-PAD

Commit message: refactor: Update board design files to version 2.
Parts:
- added U$1: RTC-DS3231-AT24C32, diy-modules:RTC-DS3231-AT24C32
- added X7: btn0, Rembrandt Electronics - JST XH Connectors v1-0:JST-XH-02-PACKAGE-LONG-PAD
- moved BTN5 22.1 mm to (48.5, 64.8)
- moved XA1 21.8 mm to (84.2, 62.8)
- moved J1 21.8 mm to (94.7, 64.6), turned to 0 degrees
- moved X5 21.6 mm to (57.6, 64.8)
- moved X6 21.2 mm to (70.0, 64.7)
- moved X8 5.38 mm to (85.1, 50.5)
- moved R1 3.74 mm to (26.8, 62.8)
- moved R2 3.70 mm to (36.9, 62.9)
- moved RTC 0.41 mm to (26.1, 49.4)
Connections:
- new net GND.1: U$1.J1.6
- new net GND.2: U$1.J2.4
- new net VCC.1: U$1.J1.5
- new net VCC.2: U$1.J2.3
- net VBUS: now also X7.1, X7.2
Routing:
- net VBUS: track 125.2 -> 174.9 mm
- net GND: track 239.5 -> 277.6 mm
- net RX2: track 44.4 -> 65.5 mm
- net TX2: track 44.0 -> 64.6 mm
- net 0: track 33.8 -> 52.3 mm
- net TX1: track 44.1 -> 59.4 mm
- net BTN: track 48.5 -> 62.9 mm
- net RX1: track 47.0 -> 60.2 mm
- net 3V3: track 70.9 -> 76.9 mm
- net SDA: track 63.7 -> 59.4 mm
- net RST: track 47.9 -> 48.8 mm, vias 2 -> 0

Commit message: feat: Create new schematic file and remove `diy-modules` library from board layout.
Parts:
- removed U$1: RTC-DS3231-AT24C32, diy-modules:RTC-DS3231-AT24C32
Connections:
- removed net GND.1: U$1.J1.6
- removed net GND.2: U$1.J2.4
- removed net VCC.1: U$1.J1.5
- removed net VCC.2: U$1.J2.3
Changed lines of the file:
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@@
 <attribute name="VALUE" x="19.5025" y="58.2075" size="1.016" layer="27" ratio="10" rot="R180"/>
-</element>
-<element name="U$1" library="diy-modules" package="RTC-DS3231-AT24C32" value="RTC-DS3231-AT24C32" x="44" y="49.3" smashed="yes" rot="R180">
-<attribute name="NAME" x="44" y="36.6" size="1.27" layer="25" rot="R180" align="bottom-center"/>
-<attribute name="VALUE" x="44" y="62" size="1.27" layer="27" rot="R180" align="top-center"/>
 </element>
 <element name="X7" library="Rembrandt Electronics - JST XH Connectors v1-0" package="JST-XH-02-PACKAGE-LONG-PAD" value="btn0" x="94.7" y="56.5" smashed="yes">
@@
 <contactref element="XA1" pad="1"/>
 </signal>
-<signal name="VCC.1">
-<contactref element="U$1" pad="J1.5"/>
-</signal>
-<signal name="GND.2">
-<contactref element="U$1" pad="J2.4"/>
-</signal>
-<signal name="VCC.2">
-<contactref element="U$1" pad="J2.3"/>
-</signal>
-<signal name="GND.1">
-<contactref element="U$1" pad="J1.6"/>
-</signal>
 </signals>
